Commit message: moveit, camera, rpi files

File: elvin/robit_ws/src/robit_urdf/urdf/robit.xacro (robot description, xacro)
@@ -28,5 +28,6 @@
 	<xacro:property name="upper_arm_l" value="0.025"/>
 	<xacro:property name="upper_arm_w" value="0.027"/>
-	<xacro:property name="upper_arm_h" value="0.145"/>
+	<!-- <xacro:property name="upper_arm_h" value="0.145"/> -->
+	<xacro:property name="upper_arm_h" value="0.12"/>
 	<xacro:property name="elbow_l" value="0.07"/>
 	<xacro:property name="elbow_w" value="0.036"/>
@@ -43,6 +44,6 @@
 	<xacro:property name="finger_r" value="0.016"/>
 	<xacro:property name="gripper_l" value="0.13"/>
-	<xacro:property name="gripper_w" value="0.115"/>
-	<xacro:property name="gripper_h" value="0.01"/>
+	<xacro:property name="gripper_w" value="0.112"/>
+	<xacro:property name="gripper_h" value="0.016"/>
 	<!-- MOI -->
 	<xacro:macro name="default_inertial" params="mass">
@@ -58,4 +59,6 @@
 				<material name="gray"/>
 			</geometry>
+			<origin rpy="0 0 0" xyz="-0.0475 0 0"/>
+			<!-- <origin rpy="0 0 0" xyz="0.0 0 0"/> -->
 			<material name="gray"/>
 		</visual>
@@ -63,5 +66,7 @@
 			<geometry>
 				<box size="${base_link_l} ${base_link_w} ${base_link_h}"/>
-			</geometry>
+				<!-- <origin rpy="0 0 0" xyz="0 0 0"/> -->
+			</geometry>
+			<origin rpy="0 0 0" xyz="-0.0475 0 0"/>
 		</collision>
 	<!--	<xacro:default_inertial mass="0.001"/> -->
@@ -83,9 +88,11 @@
 		<xacro:default_inertial mass="0.001"/>
 	</link>
+	<!-- Servo 1 -->
 	<joint name="shoulder_rotate" type="revolute">
 		<parent link="base_link"/>
 		<child link="shoulder"/>
 		<axis xyz="0 0 1"/>
-		<origin xyz="0.0125 0 0.004"/>
+		<!-- <origin xyz="0.0125 0 0.004"/> -->
+		<origin xyz="-0.035 0 0.004"/>
 		<limit effort="100.0" lower="-1.67552" upper="1.5708" velocity="10000000"/>
 	</joint>
@@ -158,5 +165,6 @@
 				<box size="${upper_arm_l} ${upper_arm_w} ${upper_arm_h}"/>
 			</geometry>
-			<origin rpy="0 0 0" xyz="0 -0.024 0.0575"/>
+			<!-- <origin rpy="0 0 0" xyz="0 -0.024 0.0575"/> -->
+			<origin rpy="0 0 0" xyz="0 -0.024 0.06"/>
 			<material name="gray"/>
 		</visual>
@@ -165,8 +173,10 @@
 				<box size="${upper_arm_l} ${upper_arm_w} ${upper_arm_h}"/>
 			</geometry>
-			<origin rpy="0 0 0" xyz="0 -0.024 0.0575"/>
-		</collision>
-		<xacro:default_inertial mass="0.001"/>
-	</link>
+			<!-- <origin rpy="0 0 0" xyz="0 -0.024 0.0575"/> -->
+			<origin rpy="0 0 0" xyz="0 -0.024 0.06"/>
+		</collision>
+		<xacro:default_inertial mass="0.001"/>
+	</link>
+	<!-- Servo 2 -->
 	<joint name="left_bracket_to_upper_arm" type="revolute">
 		<parent link="left_bracket"/>
@@ -175,4 +185,5 @@
 		<axis xyz="0 1 0"/>
 		<limit effort="100.0" lower="0" upper="2.58309" velocity="10000000"/>
+		<!-- <limit effort="100.0" lower="0" upper="2.61799" velocity="10000000"/> -->
 	</joint>
 	<link name="elbow">
@@ -192,10 +203,13 @@
 		<xacro:default_inertial mass="0.001"/>
 	</link>
+	<!-- Servo 3 -->
 	<joint name="elbow_joint" type="revolute">
 		<parent link="upper_arm"/>
 		<child link="elbow"/>
-		<origin rpy="0 1.22173 0" xyz="0 -0.024 0.125"/>
+		<!-- <origin rpy="0 1.22173 0" xyz="0 -0.024 0.125"/> -->
+		<origin rpy="0 1.22173 0" xyz="0 -0.024 0.12"/>
 		<axis xyz="0 1 0"/>
 		<limit effort="100.0" lower="-2.30383" upper="0" velocity="10000000"/>
+		<!-- <limit effort="100.0" lower="-2.25147" upper="0" velocity="10000000"/> -->
 	</joint>
 	<link name="forearm">
@@ -215,4 +229,5 @@
 		<xacro:default_inertial mass="0.001"/>
 	</link>
+	<!-- Servo 4 -->
 	<joint name="forearm_rotate" type="revolute">
 		<parent link="elbow"/>
@@ -259,4 +274,5 @@
 		<xacro:default_inertial mass="0.001"/>
 	</link>
+	<!--Servo 5 -->
 	<joint name="wrist_joint" type="revolute">
 		<parent link="wrist"/>
@@ -264,5 +280,6 @@
 		<axis xyz="0 1 0"/>
 		<origin xyz="0.035 0 0"/>
-		<limit effort="100.0" lower="-1.51536" upper="1.4784" velocity="10000000"/>
+		<!-- <limit effort="100.0" lower="-1.51536" upper="1.4784" velocity="10000000"/> -->
+		<limit effort="100.0" lower="-1.423" upper="1.571" velocity="10000000"/>
 	</joint>
 	<link name="finger">
@@ -287,7 +304,7 @@
 		<axis xyz="1 0 0"/>
 		<origin xyz="0.026 0 0"/>
-		<limit effort="100.0" lower="-1.5708" upper="1.75559" velocity="10000000"/>
-	</joint>
-	<!--
+		<!-- <limit effort="100.0" lower="-1.5708" upper="1.75559" velocity="10000000"/> -->
+		<limit effort="100.0" lower="-1.2" upper="1.2" velocity="10000000"/>
+	</joint>
  	<link name="gripper">
 		<visual>
@@ -295,5 +312,5 @@
 				<box size="${gripper_l} ${gripper_w} ${gripper_h}"/>
 			</geometry>
-			<origin xyz="0.05 0 0"/>
+			<origin xyz="0.065 0 0"/>
 		</visual>
 		<collision>
@@ -301,5 +318,5 @@
 				<box size="${gripper_l} ${gripper_w} ${gripper_h}"/>
 			</geometry>
-			<origin xyz="0.05 0 0"/>
+			<origin xyz="0.065 0 0"/>
 		</collision>
 		<xacro:default_inertial mass="0.001"/>
@@ -310,4 +327,27 @@
 		<origin xyz="0.004 0 0"/>
 	</joint>
-	-->
+	<link name="tip">
+		<visual>
+			<geometry>
+				<box size="0.01 0.01 0.01"/>
+			</geometry>
+			<material name="white"/>
+			<!-- <origin xyz="0.065 0 0"/> -->
+			<origin xyz="0.0 0 0"/>
+		</visual>
+		<collision>
+			<geometry>
+				<box size="0.01 0.01 0.01"/>
+			</geometry>
+			<!-- <origin xyz="0.065 0 0"/> -->
+			<origin xyz="0.0 0 0"/>
+		</collision>
+		<xacro:default_inertial mass="0.001"/>
+	</link>
+	<joint name="gripper_to_tip" type="fixed">
+		<parent link="gripper"/>
+		<child link="tip"/>
+		<origin xyz="0.13 0 0"/>
+		<!-- <origin xyz="0.065 0 0"/> -->
+	</joint>
 </robot>

File: elvin/robit_ws/src/robit_urdf/urdf/robit2.urdf (robot description, URDF)
Before this commit: robot robit_urdf, 11 links, 10 joints
Links:
- added link gripper, mass 0.001; collision box size=0.13 0.112 0.016; visual box size=0.13 0.112 0.016
- added link tip, mass 0.001; collision box size=0.01 0.01 0.01; visual box size=0.01 0.01 0.01
- link upper_arm: geometry collision box size=0.025 0.027 0.12; visual box size=0.025 0.027 0.12
Joints:
- added joint finger_to_gripper: type fixed, parent finger, child gripper, origin xyz=0.004 0 0
- added joint gripper_to_tip: type fixed, parent gripper, child tip, origin xyz=0.13 0 0
- joint elbow_joint: origin xyz=0 -0.024 0.125 rpy=0 1.22173 0 -> xyz=0 -0.024 0.12 rpy=0 1.22173 0
- joint finger_rotate: limit lower=-1.5708 upper=1.75559 effort=100.0 velocity=10000000 -> lower=-1.2 upper=1.2 effort=100.0 velocity=10000000
- joint shoulder_rotate: origin xyz=0.0125 0 0.004 -> xyz=-0.035 0 0.004
- joint wrist_joint: limit lower=-1.51536 upper=1.4784 effort=100.0 velocity=10000000 -> lower=-1.423 upper=1.571 effort=100.0 velocity=10000000
